Commit message: Add files

File: description/robot.urdf.xacro (robot description, xacro)
@@ -1,7 +1,6 @@
 <?xml version="1.0"?>
-<robot xmlns:xacro="http://www.ros.org/wiki/xacro"  name="robot">
+<robot xmlns:xacro="http://www.ros.org/wiki/xacro">
     <!-- Example link -->
+    <xacro:include filename="properties.xacro"/>
     <xacro:include filename="robot_core.xacro"/>
-        <!-- Example link -->
-    <link name="base_link"></link>
 </robot>

Commit message: First functional, pending controller

File: description/robot.urdf.xacro (robot description, xacro)
@@ -1,7 +1,7 @@
 <?xml version="1.0"?>
-<robot xmlns:xacro="http://www.ros.org/wiki/xacro"  name="robot">
+<robot xmlns:xacro="http://www.ros.org/wiki/xacro" name="Myrobot">
     <!-- Example link -->
     <xacro:include filename="robot_core.xacro"/>
-        <!-- Example link -->
-    <link name="base_link"></link>
+    <xacro:include filename="properties.xacro"/>
+    <xacro:include filename="gazebo_control.xacro"/>
 </robot>
