Commit message: Gazebo stuff and readme changes

File: description/robot_core.xacro (robot description, xacro)
@@ -89,3 +89,18 @@
         </collision>
     </link>
+    <!-- Gazebo stuff (remove?)-->
+    <gazebo reference="chassis">
+        <material>Gazebo/White</material>
+    </gazebo>
+    <gazebo reference="left_wheel">
+        <material>Gazebo/Blue</material>
+    </gazebo>
+    <gazebo reference="right_wheel">
+        <material>Gazebo/Blue</material>
+    </gazebo>
+    <gazebo reference="caster_wheel">
+        <material>Gazebo/Black</material>
+        <mu1 value = "0.001" />
+        <mu2 value = "0.001" />
+    </gazebo>
 </robot>

Commit message: Major change, cloned from andres branch

File: description/robot_core.xacro (robot description, xacro)
@@ -4,5 +4,5 @@
     <link name="base_link">
     </link>
-    <!-- Example link -->
+   <!-- Example link -->
     <xacro:include filename="inertial_macros.xacro"/>
     <joint name="base_link" type="fixed">
@@ -26,4 +26,7 @@
             </geometry>
         </collision>
+        <xacro:inertial_box mass="0.5" x="0.3" y="0.3" z="0.15">
+            <origin xyz="0.15 0 0.075" rpy="0 0 0"/>
+        </xacro:inertial_box>
     </link>
     <!-- left wheel joint -->
@@ -47,4 +50,7 @@
             </geometry>
         </collision>
+        <xacro:inertial_cylinder mass="0.1" length="0.04" radius="0.05">
+          <origin xyz="0 0 0" rpy="0 0 0"/>
+        </xacro:inertial_cylinder>
     </link>
     <!-- right wheel joint -->
@@ -68,4 +74,7 @@
             </geometry>
         </collision>
+        <xacro:inertial_cylinder mass="0.1" length="0.04" radius="0.05">
+            <origin xyz="0 0 0" rpy="0 0 0"/>
+        </xacro:inertial_cylinder>
     </link>
     <!-- caster wheel joint -->
@@ -75,5 +84,5 @@
         <origin xyz="0.24 0 0"/>
     </joint>
-    <!-- left wheel link -->
+    <!-- caster wheel link -->
     <link name="caster_wheel">
         <visual>
@@ -87,8 +96,10 @@
                 <sphere radius="0.05"/>
             </geometry>
+        <xacro:inertial_sphere mass="0.1" radius="0.05">
+            <origin xyz="0 0 0" rpy="0 0 0"/>
+        </xacro:inertial_sphere>
         </collision>
     </link>
-    <!-- Gazebo tags stuff (remove?) color reference tags-->
-    <gazebo reference="chassis">
+	<gazebo reference="chassis">
         <material>Gazebo/White</material>
     </gazebo>

Commit message: robot_core modified to account for changes, LIDAR FUNCTIONAL

File: description/robot_core.xacro (robot description, xacro)
@@ -47,5 +47,5 @@
         <collision>
             <geometry>
-                <cylinder radius="0.05" length="0.04"/>
+	              <sphere radius="0.05"/>
             </geometry>
         </collision>
@@ -71,5 +71,5 @@
         <collision>
             <geometry>
-                <cylinder radius="0.05" length="0.04"/>
+                <sphere radius="0.05" />
             </geometry>
         </collision>
